File: hardware/epdiy-v7/epaper-breakout.kicad_pcb (KiCad board)
At the start: 4 copper layers, 100 x 55 mm, 118 parts, among them J1 USB_C_Receptacle_USB2.0, J2 EXTENSION_HEADER, J3 USB_HDR, J4 XF2M-3315-1A, J5 CONN_BAT, J6 8BIT_HEADER, J7 ESP_HDR, Q1 AO3401A, Q3 MMBT3904, Q4 MMBT3904, U1 RT9080-33GJ5, U10 ED060XC5, U11 TP4056, U2 PCA9535PW, U3 TPS651851RSLR, U4 USBLC6-2P6, U5 XC6206PxxxMR, U6 ED078KH6, U7 PCF8563T, U8 ESP32-S3-WROOM-1, U9 CH340C, Y1 32.768K

Commit message: v7 hardware fixes
Connections:
- J7 pad 7: /GPIO_45 -> /IO0
- Q4 pad 3: /EP_STV -> /IO0
- R15 pad 1: /EP_STV -> /IO0
- U8 pad 26: /GPIO_45 -> /EP_STV
- U8 pad 27: /EP_STV -> /IO0
- U9 pad 5: /USB_D- -> /USB_D+
- U9 pad 6: /USB_D+ -> /USB_D-
Routing:
- net /IO0: track 0.00 -> 64.1 mm, vias 0 -> 5
- net /EP_STV: track 106.1 -> 57.7 mm, vias 10 -> 6
- net /GPIO_45: track 33.0 -> 0.00 mm, vias 2 -> 0
- net /USB_D+: track 13.9 -> 18.0 mm
- net /~{GPIO_INTR}: track 43.6 -> 46.5 mm
- net /EP_OE: track 89.6 -> 92.1 mm
- net /EP_MODE: track 99.1 -> 101.3 mm
- net /USB_D-: track 14.5 -> 15.2 mm
Other:
- board text added: "IO0"
- board text removed: "IO45"
