File: hardware/epdiy-v7/epaper-breakout.kicad_sch (KiCad schematic)
At the start: 117 parts, among them J1 USB_C_Receptacle_USB2.0, J2 EXTENSION_HEADER, J3 USB_HDR, J4 XF2M-3315-1A, J5 CONN_BAT, J6 8BIT_HEADER, J7 ESP_HDR, Q1 AO3401A, Q3 MMBT3904, Q4 MMBT3904, U1 RT9080-33GJ5, U10 ED060XC5, U11 TP4056, U2 PCA9535PW, U3 TPS651851RSLR, U4 USBLC6-2P6, U5 XC6206PxxxMR, U6 ED078KH6, U7 PCF8563T, U8 ESP32-S3-WROOM-1, U9 CH340C, Y1 32.768K

Commit message: v7 hardware fixes
Connections:
- net EP_STV: now also U8.26 (GPIO45); no longer Q4.3 (C), R15.1, U8.27 (GPIO0/BOOT)
- net USB_D+: now also U9.5 (UD+); no longer U9.6 (UD-)
- net USB_D-: now also U9.6 (UD-); no longer U9.5 (UD+)
- net GPIO_45 renamed IO0
- net IO0: now also Q4.3 (C), R15.1, U8.27 (GPIO0/BOOT); no longer U8.26 (GPIO45)
